Commit message: fix description issue

File: noetic_workspace/src/demo/urdf/panther_macro.urdf.xacro (robot description, xacro)
@@ -13,5 +13,5 @@
                        simulation_engine:='gazebo-classic'">
     <xacro:if value="${wheel_config_path == 'None'}">
-      <xacro:property name="wheel_config_file" value="$(find panther_description)/config/WH01.yaml"  />
+      <xacro:property name="wheel_config_file" value="$(find demo)/config/WH01.yaml"  />
     </xacro:if>
     <xacro:unless value="${wheel_config_path == 'None'}">
@@ -21,6 +21,6 @@
     <xacro:property name="wheel_config" value="${wheel_config_ros_params['/**']['ros__parameters']}" />
     <!-- INCLUDE ROBOT PARTS DEFINITIONS -->
-    <xacro:include filename="$(find panther_description)/urdf/body.urdf.xacro" ns="body" />
-    <xacro:include filename="$(find panther_description)/urdf/wheel.urdf.xacro" ns="wheel" />
+    <xacro:include filename="$(find demo)/urdf/body.urdf.xacro" ns="body" />
+    <xacro:include filename="$(find demo)/urdf/wheel.urdf.xacro" ns="wheel" />
     <!-- BODY DECLARATION -->
     <xacro:body.body

Commit message: change to rotate

File: noetic_workspace/src/demo/urdf/panther_macro.urdf.xacro (robot description, xacro)
@@ -13,5 +13,5 @@
                        simulation_engine:='gazebo-classic'">
     <xacro:if value="${wheel_config_path == 'None'}">
-      <xacro:property name="wheel_config_file" value="$(find demo)/config/WH01.yaml"  />
+      <xacro:property name="wheel_config_file" value="$(find panther_description)/config/WH01.yaml"  />
     </xacro:if>
     <xacro:unless value="${wheel_config_path == 'None'}">
@@ -21,6 +21,6 @@
     <xacro:property name="wheel_config" value="${wheel_config_ros_params['/**']['ros__parameters']}" />
     <!-- INCLUDE ROBOT PARTS DEFINITIONS -->
-    <xacro:include filename="$(find demo)/urdf/body.urdf.xacro" ns="body" />
-    <xacro:include filename="$(find demo)/urdf/wheel.urdf.xacro" ns="wheel" />
+    <xacro:include filename="$(find panther_description)/urdf/body.urdf.xacro" ns="body" />
+    <xacro:include filename="$(find panther_description)/urdf/wheel.urdf.xacro" ns="wheel" />
     <!-- BODY DECLARATION -->
     <xacro:body.body
